Commit message: Fix the encoder pin for right wheel

File: lidarbot_description/urdf/lidar.xacro (robot description, xacro)
@@ -21,5 +21,5 @@
         <parent link="base_link"/>
         <child link="lidar_link"/>
-        <origin xyz="0.1385 0.0095 0.08" rpy="0 0 ${-pi/2}"/>
+        <origin xyz="0.1385 0.0095 0.08" rpy="0 0 0"/>
         <axis xyz="0 0 1"/>
     </joint>
