Commit message: Update the gazebo files for Jazzy

File: lidarbot_gz/urdf/lidarbot_gz.urdf.xacro (robot description, xacro)
@@ -6,5 +6,5 @@
   <ros2_control name="IgnitionSystem" type="system">
     <hardware>
-      <plugin>ign_ros2_control/IgnitionSystem</plugin>
+      <plugin>gz_ros2_control/GazeboSimSystem</plugin>
     </hardware>
     <joint name="left_wheel_joint">
@@ -26,5 +26,5 @@
   </ros2_control>
   <gazebo>
-    <plugin filename="ign_ros2_control-system" name="ign_ros2_control::IgnitionROS2ControlPlugin">
+    <plugin filename="gz_ros2_control-system" name="gz_ros2_control::GazeboSimROS2ControlPlugin">
       <parameters>$(find lidarbot_bringup)/config/controllers.yaml</parameters>
     </plugin>

File: lidarbot_gz/urdf/lidarbot_gz_core.xacro (robot description, xacro)
@@ -112,5 +112,5 @@
       <!-- Rplidar base -->
       <visual name="rplidar_base_visual">
-        <origin xyz="0.13985 0.0087 0.037" rpy="0 0 ${-pi/2}"/>
+        <origin xyz="0.13985 0.0087 0.037" rpy="0 0 0"/>
           <geometry>
             <mesh filename="file://$(find lidarbot_description)/meshes/rplidar_base.dae"/>

File: lidarbot_gz/urdf/sensors.xacro (robot description, xacro)
@@ -146,5 +146,5 @@
     <parent link="base_link"/>
     <child link="lidar_link"/>
-    <origin xyz="0.1385 0.0095 0.08" rpy="0 0 ${-pi/2}"/>
+    <origin xyz="0.1385 0.0095 0.08" rpy="0 0 0"/>
     <axis xyz="0 0 1"/>
   </joint>
